Commit message: Added simulations with kinect

File: schunk_description/urdf/lwa4p/lwa4p.gazebo.xacro (robot description, xacro)
@@ -37,4 +37,47 @@
       <material value="Schunk/LightGrey" />
     </gazebo>
+    <!-- camera -->
+    <gazebo reference="camera_link">
+      <sensor type="depth" name="camera1">
+          <always_on>1</always_on>
+          <visualize>true</visualize>
+          <camera>
+              <horizontal_fov>1.047</horizontal_fov>
+              <image>
+                  <width>640</width>
+                  <height>480</height>
+                  <format>R8G8B8</format>
+              </image>
+              <depth_camera>
+              </depth_camera>
+              <clip>
+                  <near>0.1</near>
+                  <far>100</far>
+              </clip>
+          </camera>
+               <plugin name="camera_controller" filename="libgazebo_ros_openni_kinect.so">
+               <alwaysOn>true</alwaysOn>
+                  <updateRate>10.0</updateRate>
+                  <cameraName>camera</cameraName>
+                  <frameName>camera_link</frameName>
+              <imageTopicName>rgb/image_raw</imageTopicName>
+              <depthImageTopicName>depth/image_raw</depthImageTopicName>
+              <pointCloudTopicName>depth/points</pointCloudTopicName>
+              <cameraInfoTopicName>rgb/camera_info</cameraInfoTopicName>
+              <depthImageCameraInfoTopicName>depth/camera_info</depthImageCameraInfoTopicName>
+              <pointCloudCutoff>0.4</pointCloudCutoff>
+                  <hackBaseline>0.07</hackBaseline>
+                  <distortionK1>0.0</distortionK1>
+                  <distortionK2>0.0</distortionK2>
+                  <distortionK3>0.0</distortionK3>
+                  <distortionT1>0.0</distortionT1>
+                  <distortionT2>0.0</distortionT2>
+              <CxPrime>0.0</CxPrime>
+              <Cx>0.0</Cx>
+              <Cy>0.0</Cy>
+              <focalLength>0.0</focalLength>
+              </plugin>
+      </sensor>
+    </gazebo>
   </xacro:macro>
 </robot>

File: schunk_description/urdf/lwa4p/lwa4p.urdf.xacro (robot description, xacro)
@@ -237,4 +237,5 @@
       </collision>
     </link>
+    <!-- Add gripper -->
     <joint name="${name}_ee_joint" type="fixed">
       <origin xyz="0 0 0.0824" rpy="0 0 0"/>
@@ -245,4 +246,58 @@
       <xacro:default_inertial/>
     </link>
+     <!-- Kinect link -->
+    <joint name="camera_joint" type="fixed">
+      <origin xyz="${-0.08} ${0} ${0.1470}" rpy="${M_PI} ${-M_PI/2} ${M_PI}"/>
+      <parent link="${name}_6_link"/>
+      <child link="camera_link" />
+    </joint>
+    <link name="camera_link">
+      <visual>
+       <origin xyz="0 0 0" rpy="0 0 ${M_PI/2}"/>
+        <geometry>
+         <mesh filename="package://schunk_description/meshes/kinect/kinect.dae"/>
+        </geometry>
+      </visual>
+      <collision>
+        <origin xyz="0.0 0.0 0.0" rpy="0 0 0"/>
+        <geometry>
+          <box size="0.07271 0.27794 0.073"/>
+        </geometry>
+      </collision>
+      <inertial>
+        <mass value="0.564" />
+        <origin xyz="0 0 0" />
+        <inertia ixx="0.003881243" ixy="0.0" ixz="0.0"
+                 iyy="0.000498940" iyz="0.0"
+                 izz="0.003879257" />
+      </inertial>
+    </link>
+    <joint name="camera_rgb_optical_joint" type="fixed">
+      <origin xyz="0 0 0" rpy="${-M_PI/2} 0 ${-M_PI/2}" />
+      <parent link="camera_link" />
+      <child link="camera_rgb_optical_frame" />
+    </joint>
+    <link name="camera_rgb_optical_frame"/>
+    <joint name="camera_rgb_joint" type="fixed">
+      <origin xyz="-0.031 ${0.0125} -0.016" rpy="0 0 0"/>
+      <parent link="camera_link"/>
+      <child link="camera_rgb_frame"/>
+    </joint>
+    <link name="camera_rgb_frame"/>
+    <!-- The fixed joints & links below are usually published by static_transformers launched by the OpenNi launch
+         files. However, for Gazebo simulation we need them, so we add them here.
+         (Hence, don't publish them additionally!) -->
+    <joint name="camera_depth_joint" type="fixed">
+      <origin xyz="0 ${2 * 0.0125} 0" rpy="0 0 0" />
+      <parent link="camera_rgb_frame" />
+      <child link="camera_depth_frame" />
+    </joint>
+    <link name="camera_depth_frame"/>
+    <joint name="camera_depth_optical_joint" type="fixed">
+      <origin xyz="0 0 0" rpy="${-M_PI/2} 0 ${-M_PI/2}" />
+      <parent link="camera_depth_frame" />
+      <child link="camera_depth_optical_frame" />
+    </joint>
+    <link name="camera_depth_optical_frame"/>
     <!-- extensions -->
     <xacro:schunk_lwa4p_gazebo name="${name}" />
