Commit message: Fix Kinect frame and added missing gripper's joints on gazebo

File: schunk_lwa4p_moveit/urdf/lwa4p/lwa4p.gazebo.xacro (robot description, xacro)
@@ -37,4 +37,20 @@
       <material value="Schunk/LightGrey" />
     </gazebo>
+    <!-- Gripper -->
+    <gazebo reference="${name}_gripper_base_link">
+      <gravity>true</gravity>
+      <self_collide>false</self_collide>
+      <material value="Schunk/LightGrey" />
+    </gazebo>
+    <gazebo reference="${name}_gripper_finger_left_link">
+      <gravity>true</gravity>
+      <self_collide>false</self_collide>
+      <material value="Schunk/LightGrey" />
+    </gazebo>
+    <gazebo reference="${name}_gripper_finger_right_link">
+      <gravity>true</gravity>
+      <self_collide>false</self_collide>
+      <material value="Schunk/LightGrey" />
+    </gazebo>
     <!-- camera -->
     <gazebo reference="camera_link">
@@ -58,7 +74,7 @@
                <plugin name="camera_controller" filename="libgazebo_ros_openni_kinect.so">
                <alwaysOn>true</alwaysOn>
-                  <updateRate>10.0</updateRate>
+                  <updateRate>20.0</updateRate>
                   <cameraName>camera</cameraName>
-                  <frameName>camera_link</frameName>
+                  <frameName>camera_rgb_optical_frame</frameName>
               <imageTopicName>rgb/image_raw</imageTopicName>
               <depthImageTopicName>depth/image_raw</depthImageTopicName>

File: schunk_lwa4p_moveit/urdf/lwa4p/lwa4p.transmission.xacro (robot description, xacro)
@@ -9,4 +9,7 @@
     <xacro:default_transmission jname="${name}_5"/>
     <xacro:default_transmission jname="${name}_6"/>
+    <xacro:default_transmission jname="${name}_gripper_base"/>
+    <xacro:default_transmission jname="${name}_gripper_finger_left"/>
+    <xacro:default_transmission jname="${name}_gripper_finger_right"/>
   </xacro:macro>
 </robot>

File: schunk_lwa4p_moveit/urdf/lwa4p/lwa4p.urdf.xacro (robot description, xacro)
@@ -313,5 +313,5 @@
     <!-- ============================================================================= -->
     <joint name="camera_joint" type="fixed">
-      <origin xyz="${-0.056} ${0} ${0.038}" rpy="${M_PI} ${-M_PI/2} ${M_PI}"/>
+      <origin xyz="${-0.056} ${0} ${0.038}" rpy="${0} ${-M_PI/2} ${0}"/>
       <parent link="${name}_gripper_base_link"/>
       <child link="camera_link" />
@@ -338,22 +338,22 @@
       </inertial>
     </link>
-    <joint name="camera_rgb_optical_joint" type="fixed">
-      <origin xyz="0 0 0" rpy="${-M_PI/2} 0 ${-M_PI/2}" />
-      <parent link="camera_link" />
-      <child link="camera_rgb_optical_frame" />
-    </joint>
-    <link name="camera_rgb_optical_frame"/>
     <joint name="camera_rgb_joint" type="fixed">
-      <origin xyz="-0.031 ${0.0125} -0.016" rpy="0 0 0"/>
+      <origin xyz="0 -0.005 0" rpy="0 0 0" />
       <parent link="camera_link"/>
       <child link="camera_rgb_frame"/>
     </joint>
     <link name="camera_rgb_frame"/>
+    <joint name="camera_rgb_optical_joint" type="fixed">
+       <origin xyz="0 0 0" rpy="${-M_PI/2} 0 ${-M_PI/2}" />
+      <parent link="camera_rgb_frame" />
+      <child link="camera_rgb_optical_frame" />
+    </joint>
+    <link name="camera_rgb_optical_frame"/>
     <!-- The fixed joints & links below are usually published by static_transformers launched by the OpenNi launch
          files. However, for Gazebo simulation we need them, so we add them here.
          (Hence, don't publish them additionally!) -->
     <joint name="camera_depth_joint" type="fixed">
-      <origin xyz="0 ${2 * 0.0125} 0" rpy="0 0 0" />
-      <parent link="camera_rgb_frame" />
+      <origin xyz="0 0.018 0" rpy="0 0 0" />
+      <parent link="camera_link" />
       <child link="camera_depth_frame" />
     </joint>
